File: tactile_sensor/tactile_sensor.kicad_pcb (KiCad board)
At the start: 2 copper layers, 20 x 30 mm, 12 parts

Commit message: updated tactile_sensor design
Parts:
- moved AOUT 0.13 mm to (58.8, 74.2)
- moved DIN 0.13 mm to (59.3, 69.8)
- moved R1 0.13 mm to (58.8, 77.1)
- moved R10 0.13 mm to (63.8, 77.1)
- moved R2 0.13 mm to (59.8, 77.1)
- moved R3 0.13 mm to (60.8, 77.1)
- moved R4 0.13 mm to (61.8, 77.1)
- moved R5 0.13 mm to (62.8, 77.1)
- moved R6 0.13 mm to (67.8, 77.1)
- moved R7 0.13 mm to (66.8, 77.1)
- moved R8 0.13 mm to (65.8, 77.1)
- moved R9 0.13 mm to (64.8, 77.1)
Routing:
- net (no net): vias 110 -> 112
